Commit message: added circular trajectory dataset

File: simulation/models/clusters_urdf/strawberry_cluster.urdf (robot description, URDF)
Before this commit: robot strawberry_plant, 6 links, 5 joints
Links:
- link Upperstem: mass None -> 0.0
- link inner_jointlink_1: mass None -> 0.0
- link inner_jointlink_2: mass None -> 0.0
